Commit message: upgrading the sensor

File: catkin_ws/src/my_robot/urdf/my_robot.xacro (robot description, xacro)
@@ -132,12 +132,12 @@
     </visual>
   </link>
-  <joint type="fixed" name="camera_joint">
-    <origin xyz="0.4 0 0" rpy="0 0 0"/>
+ <joint type="fixed" name="camera_joint">
+    <origin xyz="0.4 0 0" rpy="-1.5707 0 -1.5707"/>
     <axis xyz="0 1 0"/>
-    <child link="camera"/>
+    <child link="camera_link_optical"/>
     <parent link="chassis"/>
   </joint>
-  <link name ="camera">
-    <origin xyz="0 0 0" rpy="0 0 0"/>
+   <link name ="camera_link_optical">
+    <origin xyz="0 0 0" rpy="0 1.5707 0"/>
     <geometry>
       <box size="0.05 0.05 0.05"/>

Commit message: upgrading sensor

File: catkin_ws/src/my_robot/urdf/my_robot.xacro (robot description, xacro)
@@ -133,5 +133,5 @@
   </link>
  <joint type="fixed" name="camera_joint">
-    <origin xyz="0.4 0 0" rpy="-1.5707 0 -1.5707"/>
+    <origin xyz="0.4 0 0" rpy="0 0 0"/>
     <axis xyz="0 1 0"/>
     <child link="camera_link_optical"/>

Commit message: fixed the pointcloud issue

File: catkin_ws/src/my_robot/urdf/my_robot.xacro (robot description, xacro)
@@ -132,12 +132,12 @@
     </visual>
   </link>
- <joint type="fixed" name="camera_joint">
+  <joint type="fixed" name="camera_joint">
     <origin xyz="0.4 0 0" rpy="0 0 0"/>
     <axis xyz="0 1 0"/>
-    <child link="camera_link_optical"/>
-    <parent link="chassis"/>
-  </joint>
-   <link name ="camera_link_optical">
-    <origin xyz="0 0 0" rpy="0 1.5707 0"/>
+    <child link="camera"/>
+    <parent link="chassis"/>
+  </joint>
+  <link name ="camera">
+    <origin xyz="0 0 0" rpy="0 0 0"/>
     <geometry>
       <box size="0.05 0.05 0.05"/>
@@ -164,4 +164,11 @@
       </geometry>
     </visual>
+  </link>
+  <joint name="camera_optical_joint" type="fixed">
+    <origin xyz="0 0 0" rpy="-1.5707 0 -1.5707"/>
+    <parent link="camera"/>
+    <child link="camera_link_optical"/>
+  </joint>
+  <link name="camera_link_optical">
   </link>
   <joint type="fixed" name="hokuyo_joint">
